File: batradio_pcb/rpisdr/PREAMP.kicad_sch (KiCad schematic)
At the start: 32 parts, among them U5 lmh6629, U6 lmh6629

Commit message: Corrected schematic and added mykicadlibs
Parts:
- removed RV1: 2k2, Potentiometer_SMD:Potentiometer_Bourns_3214J_Horizontal, symbol rpisdr-rescue:R_POT-Device
- removed U5, U6: lmh6629, Package_TO_SOT_SMD:SOT-23-5, symbol rpisdr-rescue:lmh6629-mylib
- added RV1: R_Pot, Potentiometer_SMD:Potentiometer_Bourns_3214J_Horizontal, symbol Device:R_Potentiometer
- added U5, U6: lmh6629, Package_TO_SOT_SMD:SOT-23-5, symbol mylibxx:lmh6629
- C10, C13, C14, C15, C16, C17, C18, C19, C20, C21: footprint Capacitor_SMD:C_0805_2012Metric_Pad1.15x1.40mm_HandSolder -> Capacitor_SMD:C_0805_2012Metric_Pad1.18x1.45mm_HandSolder
- C11, C12, C22, C25, C9: footprint Capacitor_SMD:C_1206_3216Metric_Pad1.42x1.75mm_HandSolder -> Capacitor_SMD:C_1206_3216Metric_Pad1.33x1.80mm_HandSolder
- R10, R11, R12, R13, R14, R7, R8, R9: footprint Resistor_SMD:R_0805_2012Metric_Pad1.15x1.40mm_HandSolder -> Resistor_SMD:R_0805_2012Metric_Pad1.20x1.40mm_HandSolder
Connections:
- net GND: now also RV1.3, U5.2 (V-), U6.2 (V-)
- net Sout: now also U6.1 (Out)
- net V4.5A: now also U6.5 (V+)
- net at C11.1, R10.1: now also U5.1 (Out)
- net at C10.1, R7.2, R8.1: now also U5.3 (In+)
- net at R10.2, R9.1: now also U5.4 (In-)
- net at C22.1, L6.1, R7.1: now also U5.5 (V+)
- net at C13.1, R11.2, R12.1: now also U6.3 (In+)
- net at R13.1, R14.2: now also U6.4 (In-)
- net at C11.2: now also RV1.1
- net at C14.1, C15.1, C16.2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: now also RV1.2

Commit message: Corrected mylib library settings
Parts:
- U5, U6: symbol mylibxx:lmh6629 -> mylib:lmh6629
Changed lines of the file:
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@@
 	)
 	(symbol
-		(lib_id "mylibxx:lmh6629")
+		(lib_id "mylib:lmh6629")
 		(at 90.17 50.8 0)
 		(unit 1)
@@
 	)
 	(symbol
-		(lib_id "mylibxx:lmh6629")
+		(lib_id "mylib:lmh6629")
 		(at 227.33 52.07 0)
 		(unit 1)
