File: batradio_pcb/rpisdr/rpisdr.kicad_pcb (KiCad board)
At the start: 2 copper layers, 65 x 56 mm, 71 parts, among them J1 RPI_header, J2 Conn_01x03, J3 Conn_01x03, U1 ldln025, U2 mcp33131, U3 ldln025, U4 ths4521, U5 lmh6629, U6 lmh6629, U7 ldln025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

Commit message: Updated README
Other:
- net class Default removed
- net class Power removed

Commit message: Corrected schematic and added mykicadlibs
Parts:
- added C27: 1u, Capacitor_SMD:C_1206_3216Metric_Pad1.33x1.80mm_HandSolder, F.Cu at (239.9, 118.9)
- C10, C13, C14, C15, C16, C17, C18, C19, C20, C21, C26, C3, C4: footprint Capacitor_SMD:C_0805_2012Metric_Pad1.15x1.40mm_HandSolder -> Capacitor_SMD:C_0805_2012Metric_Pad1.18x1.45mm_HandSolder
- C11, C12, C22, C23, C24, C25, C5, C6, C7, C8, C9: footprint Capacitor_SMD:C_1206_3216Metric_Pad1.42x1.75mm_HandSolder -> Capacitor_SMD:C_1206_3216Metric_Pad1.33x1.80mm_HandSolder
- J1: footprint Connector_PinSocket_2.54mm:PinSocket_2x20_P2.54mm_Vertical -> Connector_PinHeader_2.54mm:PinHeader_2x20_P2.54mm_Vertical; moved to F.Cu
- R1, R10, R11, R12, R13, R14, R15, R2, R3, R4, R5, R6, R7, R8, R9: footprint Resistor_SMD:R_0805_2012Metric_Pad1.15x1.40mm_HandSolder -> Resistor_SMD:R_0805_2012Metric_Pad1.20x1.40mm_HandSolder
- RV1: value 2k2 -> R_Pot
- U2: value mcp33131 -> ldln025; footprint Package_SO:MSOP-10_3x3mm_P0.5mm -> Package_TO_SOT_SMD:SOT-23-5
- U3: value ldln025 -> mcp33131; footprint Package_TO_SOT_SMD:SOT-23-5 -> library:MSOP-10_3x3mm_P0.5mm
- U4: footprint Package_SO:VSSOP-8_3.0x3.0mm_P0.65mm -> library:VSSOP-8_3x3mm_P0.65mm
- moved R4 11.0 mm to (250.7, 112.4)
- moved R5 7.07 mm to (241.4, 112.4), turned to 180 degrees
- moved U3 6.75 mm to (241.6, 104.7)
- moved U2 6.57 mm to (248.2, 104.1)
- moved C6 6.29 mm to (256.1, 112.4)
- moved C5 3.19 mm to (256.4, 116.0)
- moved R6 2.22 mm to (246.3, 112.3), turned to 0 degrees
- moved R3 1.89 mm to (250.0, 116.0)
- moved U4 0.14 mm to (241.1, 115.8)
- moved C14 0.11 mm to (213.7, 120.4)
- moved U5 0.11 mm to (209.4, 137.5)
- turned J1 to 90 degrees
Connections:
- C2 pad 1: Net-(C2-Pad1) -> Net-(U3-Vref)
- C3 pad 1: Net-(C3-Pad1) -> Net-(U3-Ain+)
- C4 pad 1: Net-(C4-Pad1) -> Net-(U3-Ain-)
- C8 pad 1: Net-(C8-Pad1) -> Net-(U2-Vout)
- J1 pad 1: Net-(J1-Pad1) -> unconnected-(J1-Pin_1-Pad1)
- J1 pad 17: Net-(J1-Pad17) -> unconnected-(J1-Pin_17-Pad17)
- L2 pad 2: Net-(C2-Pad1) -> Net-(U3-Vref)
- L3 pad 1: Net-(C2-Pad1) -> Net-(U3-Vref)
- R1 pad 1: Net-(C3-Pad1) -> Net-(U3-Ain+)
- R2 pad 1: Net-(C4-Pad1) -> Net-(U3-Ain-)
- R3 pad 1: Net-(R3-Pad1) -> Net-(U4-Vin-)
- R4 pad 1: Net-(R4-Pad1) -> Net-(U4-Vin+)
- R5 pad 2: Net-(R3-Pad1) -> Net-(U4-Vin-)
- R6 pad 2: Net-(R4-Pad1) -> Net-(U4-Vin+)
- TP5 pad 1: Net-(C3-Pad1) -> Net-(U3-Ain+)
- TP6 pad 1: Net-(C4-Pad1) -> Net-(U3-Ain-)
- U1 pad 4: Net-(U1-Pad4) -> unconnected-(U1-NC-Pad4)
- U2 pad 1: Net-(C2-Pad1) -> /ADC_SPI/4.5Volt
- U2 pad 2: Net-(C8-Pad1) -> GND
- U2 pad 3: Net-(C3-Pad1) -> /ADC_SPI/4.5Volt
- U2 pad 4: Net-(C4-Pad1) -> unconnected-(U2-NC-Pad4)
- U2 pad 5: GND -> Net-(U2-Vout)
- U3 pad 1: /ADC_SPI/4.5Volt -> Net-(U3-Vref)
- U3 pad 2: GND -> Net-(U2-Vout)
- U3 pad 3: /ADC_SPI/4.5Volt -> Net-(U3-Ain+)
- U3 pad 4: Net-(U3-Pad4) -> Net-(U3-Ain-)
- U3 pad 5: Net-(C8-Pad1) -> GND
- U4 pad 1: Net-(R4-Pad1) -> Net-(U4-Vin-)
- U4 pad 8: Net-(R3-Pad1) -> Net-(U4-Vin+)
- U7 pad 4: Net-(U7-Pad4) -> unconnected-(U7-NC-Pad4)
Routing:
- net Net-(U3-Vref): track 0.00 -> 30.7 mm
- net Net-(C2-Pad1): track 30.7 -> 0.00 mm
- net Net-(U2-Vout): track 0.00 -> 19.4 mm
- net Net-(C8-Pad1): track 19.4 -> 0.00 mm
- net Net-(U3-Ain-): track 0.00 -> 16.7 mm
- net Net-(C4-Pad1): track 16.7 -> 0.00 mm
- net Net-(U4-Vout-): track 26.4 -> 11.0 mm
- net Net-(U4-Vin-): track 0.00 -> 15.4 mm, vias 0 -> 2
- net Net-(U4-Vocm): track 0.00 -> 14.9 mm
- net Net-(U3-Ain+): track 0.00 -> 13.6 mm
- net Net-(C3-Pad1): track 13.6 -> 0.00 mm
- net Net-(R3-Pad1): track 9.26 -> 0.00 mm
- net Net-(U4-Vout+): track 18.8 -> 10.8 mm
- net Net-(U4-Vin+): track 0.00 -> 7.88 mm
- net Net-(R4-Pad1): track 7.73 -> 0.00 mm
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